File: pcb/atfblast.kicad_pcb (KiCad board)
At the start: 2 copper layers, 88.8 x 42.8 mm, 36 parts, among them J1 DS-210, J2 DIP20-panel, J3 DIP24-panel, J4 DB25_Male, Q1 BC547, Q2 BC557, SW1 SW_DIP_x01, U1 L7812, U2 L7805, U3 LM350

Commit message: add pcb rev.A1
Parts:
- Q1, Q2: footprint Package_TO_SOT_THT:TO-92_Inline -> Package_TO_SOT_THT:TO-92
- moved R9 7.81 mm to (144.2, 110.4), turned to 0 degrees
Connections:
- R9 pad 1: Net-(R9-Pad1) -> Net-(C4-Pad1)
- R9 pad 2: Net-(C4-Pad1) -> Net-(R9-Pad2)
- RV1 pad 3: Net-(C4-Pad1) -> Net-(R9-Pad2)
- U3 pad 1: Net-(R9-Pad1) -> Net-(R9-Pad2)
Routing:
- net Net-(R9-Pad2): track 0.00 -> 25.5 mm
- net Net-(R9-Pad1): track 19.4 -> 0.00 mm
- net Net-(C4-Pad1): track 36.9 -> 34.5 mm
- net GND: track 270.3 -> 268.8 mm
- net Net-(Q1-Pad2): track 14.4 -> 15.6 mm
- net Net-(Q2-Pad2): track 11.2 -> 11.8 mm
Other:
- net class Default removed
- board text added: "Rev.A1"
- board text removed: "Rev.A"
